Commit message: 多智能体共享policy跑通并补充测试流程

File: catkin_ws/src/multi_robot_scenario/xacro/p3dx/pioneer3dx.xacro (robot description, xacro)
@@ -3,9 +3,16 @@
   <xacro:arg name="velodyne_name" default="velodyne"/>
   <xacro:arg name="velodyne_topic" default="/velodyne_points"/>
+  <xacro:arg name="robot_namespace" default=""/>
+  <xacro:arg name="tf_prefix" default=""/>
+  <xacro:property name="robot_namespace" value="$(arg robot_namespace)"/>
+  <xacro:property name="tf_prefix" value="$(arg tf_prefix)"/>
   <!-- Import Rviz colors -->
   <xacro:include filename="$(find multi_robot_scenario)/xacro/materials.xacro" />
   <!-- Import robot -->
   <xacro:include filename="$(find multi_robot_scenario)/xacro/p3dx/pioneer3dx_body.xacro"/>
-  <xacro:pioneer3dx_body name="chassis" parent="base_link" meshes="package://gazebo_plugins/test/multi_robot_scenario/meshes/p3dx"/>
+  <xacro:pioneer3dx_body
+    name="chassis"
+    parent="base_link"
+    meshes="package://gazebo_plugins/test/multi_robot_scenario/meshes/p3dx"/>
   <!-- Laser -->
   <xacro:include filename="$(find multi_robot_scenario)/xacro/laser/hokuyo.xacro"/>

File: catkin_ws/src/multi_robot_scenario/xacro/p3dx/pioneer3dx_plugins.xacro (robot description, xacro)
@@ -4,5 +4,5 @@
     <gazebo>
         <plugin name="joint_state_publisher" filename="libgazebo_ros_joint_state_publisher.so">
-          <robotNamespace></robotNamespace>
+          <robotNamespace>${robot_namespace}</robotNamespace>
           <jointName>chassis_swivel_joint, swivel_wheel_joint, left_hub_joint, right_hub_joint</jointName>
           <updateRate>50.0</updateRate>
@@ -15,5 +15,6 @@
         <plugin name="differential_drive_controller" filename="libgazebo_ros_diff_drive.so">
             <rosDebugLevel>Debug</rosDebugLevel>
-            <robotNamespace></robotNamespace>
+            <robotNamespace>${robot_namespace}</robotNamespace>
+            <tf_prefix>${tf_prefix}</tf_prefix>
             <publishWheelTF>false</publishWheelTF>
             <publishWheelJointState>true</publishWheelJointState>
